Commit message: planning scene done

File: meca500_robot/urdf/robot.ros2_control.xacro (robot description, xacro)
@@ -1,8 +1,10 @@
 <?xml version="1.0"?>
 <robot xmlns:xacro="http://www.ros.org/wiki/xacro">
-  <xacro:macro name="meca500_ros2_control" params="name prefix use_mock_hardware">
+  <xacro:macro name="meca500_ros2_control" params="name prefix use_mock_hardware joint_offsets_file initial_positions_file">
     <xacro:arg name="robot_ip" default="192.168.0.100"/>
     <xacro:arg name="control_port" default="10000"/>
     <xacro:arg name="monitoring_port" default="10001"/>
+    <xacro:property name="offsets" value="${xacro.load_yaml(joint_offsets_file)}"/>
+    <xacro:property name="initial_positions" value="${xacro.load_yaml(initial_positions_file)['initial_positions']}"/>
     <ros2_control name="${name}" type="system">
       <!-- Real hardware -->
@@ -13,4 +15,10 @@
           <param name="control_port">$(arg control_port)</param>
           <param name="monitoring_port">$(arg monitoring_port)</param>
+          <param name="joint1_offset_deg">${offsets['joint1']}</param>
+          <param name="joint2_offset_deg">${offsets['joint2']}</param>
+          <param name="joint3_offset_deg">${offsets['joint3']}</param>
+          <param name="joint4_offset_deg">${offsets['joint4']}</param>
+          <param name="joint5_offset_deg">${offsets['joint5']}</param>
+          <param name="joint6_offset_deg">${offsets['joint6']}</param>
         </hardware>
       </xacro:unless>
@@ -24,30 +32,42 @@
       <joint name="${prefix}joint1">
         <command_interface name="position"/>
-        <state_interface name="position"/>
+        <state_interface name="position">
+          <param name="initial_value">${initial_positions['joint1']}</param>
+        </state_interface>
         <state_interface name="velocity"/>
       </joint>
       <joint name="${prefix}joint2">
         <command_interface name="position"/>
-        <state_interface name="position"/>
+        <state_interface name="position">
+          <param name="initial_value">${initial_positions['joint2']}</param>
+        </state_interface>
         <state_interface name="velocity"/>
       </joint>
       <joint name="${prefix}joint3">
         <command_interface name="position"/>
-        <state_interface name="position"/>
+        <state_interface name="position">
+          <param name="initial_value">${initial_positions['joint3']}</param>
+        </state_interface>
         <state_interface name="velocity"/>
       </joint>
       <joint name="${prefix}joint4">
         <command_interface name="position"/>
-        <state_interface name="position"/>
+        <state_interface name="position">
+          <param name="initial_value">${initial_positions['joint4']}</param>
+        </state_interface>
         <state_interface name="velocity"/>
       </joint>
       <joint name="${prefix}joint5">
         <command_interface name="position"/>
-        <state_interface name="position"/>
+        <state_interface name="position">
+          <param name="initial_value">${initial_positions['joint5']}</param>
+        </state_interface>
         <state_interface name="velocity"/>
       </joint>
       <joint name="${prefix}joint6">
         <command_interface name="position"/>
-        <state_interface name="position"/>
+        <state_interface name="position">
+          <param name="initial_value">${initial_positions['joint6']}</param>
+        </state_interface>
         <state_interface name="velocity"/>
       </joint>

File: meca500_robot/urdf/robot.urdf.xacro (robot description, xacro)
@@ -4,6 +4,10 @@
 <robot name="meca500" xmlns:xacro="http://www.ros.org/wiki/xacro">
   <xacro:arg name="use_mock_hardware" default="true"/>
+  <xacro:arg name="joint_offsets_file" default="$(find meca500_moveit)/config/joint_offsets.yaml"/>
+  <xacro:arg name="initial_positions_file" default="$(find meca500_moveit)/config/initial_positions.yaml"/>
   <xacro:include filename="$(find mecha500_robot)/urdf/robot.ros2_control.xacro" />
-  <xacro:meca500_ros2_control name="meca500" prefix="" use_mock_hardware="$(arg use_mock_hardware)"/>
+  <xacro:meca500_ros2_control name="meca500" prefix="" use_mock_hardware="$(arg use_mock_hardware)"
+    joint_offsets_file="$(arg joint_offsets_file)"
+    initial_positions_file="$(arg initial_positions_file)"/>
   <!-- Link link_0__base -->
   <link name="link_0__base">
